File: rx02-emulator-mega-shield.kicad_pcb (KiCad board)
At the start: 2 copper layers, 99.1 x 71.1 mm, 58 parts, among them J1 Conn_02x20_Odd_Even, P1 Digital, P2 Power, P3 Analog, P4 Analog, P5 PWM, P6 PWM, P7 Communication, Q1 2N7000, Q2 2N7000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

Commit message: Update to v1.1 board
Connections:
- U1 pad 10: /26 -> /3(**)
- U1 pad 12: /22 -> /2(**)
Routing:
- net /2(**): track 0.00 -> 34.1 mm
- net /3(**): track 0.00 -> 30.8 mm
- net /26: track 22.3 -> 0.00 mm
- net /22: track 15.1 -> 0.00 mm
Other:
- board text added: "RX02 Emulator Mega LCD Shield v1.1"
- board text removed: "RX02 Emulator Mega LCD Shield v1.0"
