File: rx02-emulator-mega-shield.sch (KiCad schematic (older format))
At the start: 58 parts, among them J1 Conn_02x20_Odd_Even, P1 Digital, P2 Power, P3 Analog, P4 Analog, P5 PWM, P6 PWM, P7 Communication, Q1 2N7000, Q2 2N7000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

Commit message: Update to v1.1 board
Connections:
- net 2(**): now also U1.12
- net 22: no longer U1.12
- net 26: no longer U1.10
- net 3(**): now also U1.10
Changed lines of the file:
@@
 Sheet 1 1
 Title ""
-Date "2022-09-05"
-Rev "Rev 1.0"
+Date "2023-03-13"
+Rev "Rev 1.1"
 Comp ""
 Comment1 ""
@@
 Text Label 7750 2350 0    60   ~ 0
 28
-Text Label 7750 1650 0    60   ~ 0
-26
 Text Label 7750 2700 0    60   ~ 0
 24
-Text Label 7750 1300 0    60   ~ 0
-22
 Text Label 1150 2000 2    60   ~ 0
 10(**)
@@
 Text Notes 7750 6500 0    50   ~ 0
 Value\n\n390\n120\n\n\n\n\n\n180\n390\n180\n390\n\n\n\n\n\n390\n\n\n180\n390\n
+Text Label 7750 1300 0    60   ~ 0
+2(**)
+Text Label 7750 1650 0    60   ~ 0
+3(**)
 $EndSCHEMATC
